File: dabao_v3c.kicad_pcb (KiCad board)
At the start: 6 copper layers, 17.8 x 21.1 mm, 67 parts, among them J1 USB_C_Receptacle_USB2.0_16P, Q1 LP0404N3T5G, Q2 LN237N3T5G, SW1 SKTAAAE010, SW2 SKTAAAE010, U1 baochip1x, U3 SMD IC PMIC;DCDC Buck-ADJ-1A,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, U4 XIAO-HALF-HOLE-23P, U5 EMS4000RSW, U7 SGM40567-4.2XG/TR, U8 SX1801CCR, U9 SMD IC PMIC;DCDC Buck-ADJ-1A,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, Y2 48.000MHz

Commit message: prettier SCH
Routing:
- net VSYS: vias 7 -> 8
Other:
- board text added: "xiao bao (小保) v1"
- board text removed: "xiao bao v1"
Changed lines of the file:
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@@
 	)
 	(gr_text "BAT"
-		(at 133 77.2 0)
+		(at 134.84 74.06 90)
 		(layer "B.SilkS")
 		(effects
@@
 		)
 	)
-	(gr_text "xiao bao v1"
-		(at 132 78.7 0)
+	(gr_text "xiao bao (小保) v1"
+		(at 131.74 78.68 0)
 		(layer "B.SilkS")
 		(effects
 			(font
 				(size 0.75 0.75)
-				(thickness 0.15)
+				(thickness 0.13)
 				(bold yes)
 			)
@@
 	)
 	(segment
-		(start 135.6 63.3)
-		(end 135.2 62.9)
-		(width 0.0889)
-		(layer "F.Cu")
-		(net 65)
-	)
-	(segment
 		(start 135.275 74.65)
 		(end 134.85 75.075)
@@
 	)
 	(segment
-		(start 135.2 62.9)
-		(end 126.7 62.9)
-		(width 0.0889)
-		(layer "F.Cu")
-		(net 65)
-	)
-	(segment
 		(start 135.48 74.65)
 		(end 135.275 74.65)
@@
 	)
 	(segment
-		(start 126.225 62.425)
-		(end 126.225 61.125)
-		(width 0.0889)
-		(layer "F.Cu")
-		(net 65)
-	)
-	(segment
 		(start 134.512803 75.437803)
 		(end 134.5 75.425)
@@
 		(net 65)
 	)
-	(segment
-		(start 126.7 62.9)
-		(end 126.225 62.425)
-		(width 0.0889)
-		(layer "F.Cu")
+	(via
+		(at 126.22 61.14)
+		(size 0.3556)
+		(drill 0.2032)
+		(layers "F.Cu" "B.Cu")
 		(net 65)
 	)
@@
 		(net 65)
 	)
+	(segment
+		(start 135.6 63.3)
+		(end 135.2 62.9)
+		(width 0.0889)
+		(layer "In2.Cu")
+		(net 65)
+	)
+	(segment
+		(start 126.225 61.125)
+		(end 126.225 61.135)
+		(width 0.0889)
+		(layer "In2.Cu")
+		(net 65)
+	)
+	(segment
+		(start 135.2 62.9)
+		(end 126.7 62.9)
+		(width 0.0889)
+		(layer "In2.Cu")
+		(net 65)
+	)
+	(segment
+		(start 126.225 62.425)
+		(end 126.225 61.125)
+		(width 0.0889)
+		(layer "In2.Cu")
+		(net 65)
+	)
+	(segment
+		(start 126.225 61.135)
+		(end 126.22 61.14)
+		(width 0.0889)
+		(layer "In2.Cu")
+		(net 65)
+	)
+	(segment
+		(start 126.7 62.9)
+		(end 126.225 62.425)
+		(width 0.0889)
+		(layer "In2.Cu")
+		(net 65)
+	)
