File: dabao_v3c.kicad_pcb (KiCad board)
At the start: 6 copper layers, 17.8 x 21.1 mm, 69 parts, among them J1 USB_C_Receptacle_USB2.0_16P, Q1 LP0404N3T5G, Q2 LN237N3T5G, SW1 SKTAAAE010, SW2 SKTAAAE010, U1 baochip1x, U3 SMD IC PMIC;DCDC Buck-ADJ-1A,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, U4 XIAO-HALF-HOLE-23P, U5 EMS4000RSW, U7 SGM40567-4.2XG/TR, U8 SX1801CCR, U9 SMD IC PMIC;DCDC Buck-ADJ-1A,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, Y2 48.000MHz

Commit message: part numbers
Parts:
- C14, C17, C19, C21: footprint Capacitor_SMD:C_0201_0603Metric -> Capacitor_SMD:C_0402_1005Metric
- moved C14 2.07 mm to (135.1, 76.6)
- moved C20 1.61 mm to (133.9, 70.2)
- moved C17 1.55 mm to (133.2, 76.6)
- moved C19 0.80 mm to (134.6, 73.2), turned to 180 degrees
- moved C21 0.36 mm to (133.9, 72.2)
- moved L1 0.32 mm to (133.7, 74.3)
- moved L3 0.25 mm to (134.9, 71.1)
- moved C16 0.16 mm to (133.1, 75.7)
- moved R15 0.10 mm to (136.0, 73.2)
Routing:
- net GND: track 9.05 -> 11.2 mm, vias 31 -> 30
- net +0.9V: track 9.24 -> 10.6 mm
- net Net-(SW1-B0): track 8.20 -> 8.78 mm
- net VSYS: track 20.5 -> 21.0 mm
