File: dabao_v3c.kicad_pcb (KiCad board)
At the start: 6 copper layers, 17.8 x 21.1 mm, 69 parts, among them J1 USB_C_Receptacle_USB2.0_16P, Q1 LP0404N3T5G, Q2 LN237N3T5G, SW1 SKTAAAE010, SW2 SKTAAAE010, U1 baochip1x, U3 SMD IC PMIC;DCDC Buck-ADJ-1A,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, U4 XIAO-HALF-HOLE-23P, U5 EMS4000RSW, U7 SGM40567-4.2XG/TR, U8 SX1801CCR, U9 SMD IC PMIC;DCDC Buck-ADJ-1A,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, Y2 48.000MHz

Commit message: more updates
Parts:
- D2: value LMBR4010BST5G -> PSBD2FD40V1H
- U5: value EMS4000RSW -> SGM7222YWQ10/TR
- U8: value SX1801CCR -> TPS22916CYFPR
- moved G*** 1.10 mm to (131.8, 62.8)
Connections:
- SW2 pad 3: /PC13 -> /PC13/BOOT
- SW2 pad 4: /PC13 -> /PC13/BOOT
- U1 pad D1: /PC13 -> /PC13/BOOT
Routing:
- net GND: track 11.2 -> 15.6 mm, vias 29 -> 37
- net VBUS: track 26.8 -> 28.1 mm
- net /PA7/ADC3: track 20.6 -> 19.8 mm
- net +3.3V: track 13.3 -> 13.8 mm, vias 11 -> 13
- net VSYS: track 21.0 -> 21.6 mm
- net /PB1: track 11.5 -> 12.0 mm
