File: dabao_v3c.kicad_sch (KiCad schematic)
At the start: 67 parts, among them J1 USB_C_Receptacle_USB2.0_16P, Q1 LP0404N3T5G, Q2 LN237N3T5G, SW1 SKTAAAE010, SW2 SKTAAAE010, U1 baochip1x, U3 SMD IC PMIC;DCDC Buck-ADJ-1A,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, U4 XIAO-HALF-HOLE-23P, U5 EMS4000RSW, U7 SGM40567-4.2XG/TR, U8 SX1801CCR, U9 SMD IC PMIC;DCDC Buck-ADJ-1A,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, Y2 48.000MHz

Commit message: part numbers
Parts:
- C14, C17, C19, C21: footprint Capacitor_SMD:C_0201_0603Metric -> Capacitor_SMD:C_0402_1005Metric
Changed lines of the file:
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@@
 			)
 		)
-		(property "Footprint" "Capacitor_SMD:C_0201_0603Metric"
+		(property "Footprint" "Capacitor_SMD:C_0402_1005Metric"
 			(at 285.115 172.72 0)
 			(effects
@@
 			)
 		)
-		(property "Footprint" "Capacitor_SMD:C_0201_0603Metric"
+		(property "Footprint" "Capacitor_SMD:C_0402_1005Metric"
 			(at 213.995 172.72 0)
 			(effects
@@
 			)
 		)
-		(property "Footprint" "Capacitor_SMD:C_0201_0603Metric"
+		(property "Footprint" "Capacitor_SMD:C_0402_1005Metric"
 			(at 199.39 173.99 0)
 			(effects
@@
 			)
 		)
-		(property "Footprint" "Capacitor_SMD:C_0201_0603Metric"
+		(property "Footprint" "Capacitor_SMD:C_0402_1005Metric"
 			(at 129.54 173.99 0)
 			(effects
