File: dabao_v3c.kicad_sch (KiCad schematic)
At the start: 67 parts, among them J1 USB_C_Receptacle_USB2.0_16P, Q1 LP0404N3T5G, Q2 LN237N3T5G, SW1 SKTAAAE010, SW2 SKTAAAE010, U1 baochip1x, U3 SMD IC PMIC;DCDC Buck-ADJ-1A,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, U4 XIAO-HALF-HOLE-23P, U5 EMS4000RSW, U7 SGM40567-4.2XG/TR, U8 SX1801CCR, U9 SMD IC PMIC;DCDC Buck-ADJ-1A,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, Y2 48.000MHz

Commit message: more updates
Parts:
- added D5, D6: B74121U0055M060, xiao:ESD-0201, symbol Seeed_libdb:Diode/DF2B7ASL,L3F
- added D7, D8: DF2B7ASL,L3F, Diode:ESD-0201, symbol Seeed_libdb:Diode/DF2B7ASL,L3F
- added R8: 5.1k, 1%, Resistor_SMD:R_0201_0603Metric, symbol power-altium-import:root_1_Res1
- added U2: TPS22916CYFPR, xiao:WLCSP4-0.4-0.77X0.77X0.33MM, symbol Seeed_libdb:Ic/SX1801CCR
- D2: value LMBR4010BST5G -> PSBD2FD40V1H; MPN LMBR4010BST5G -> PSBD2FD40V1H; Manufacturer LRC -> (none); SKU 304021082 -> (none)
- U5: value EMS4000RSW -> SGM7222YWQ10/TR; LCSC C49186227 -> C700326
- U8: value SX1801CCR -> TPS22916CYFPR; MPN SX1801CCR -> TPS22916CYFPR; Manufacturer 6SIGMA -> TI; SKU SX1801CCR -> TPS22916CYFPR; Status XIAO RP2350 -> (none)
Connections:
- net +3.3V: now also R8.1
- net GND: now also D5.1, D6.1, D7.1, D8.1, U2.B1 (GND)
- net PC13: now also R8.2; no longer SW2.3 (B0), SW2.4 (B1), U1.D1 (PC13)
- net USBCONN_N: now also D6.2
- net USBCONN_P: now also D5.2
- net VBUS: now also D8.2
- net VSYS: now also U2.A2 (VIN); no longer D1.4 (VDD)
- net PB3 renamed PB3/WS2812_PWR_EN
- net PB3/WS2812_PWR_EN: now also U2.B2 (EN)
- new net: D1.4 (VDD), U2.A1 (VOUT)
- new net PC13/BOOT: D7.2, SW2.3 (B0), SW2.4 (B1), U1.D1 (PC13)
Other:
- note added: "Indicator LEDs"
- note added: "User Input Buttons"
- note removed: "User Inputs & LEDs"
- moved on the sheet: C13, C14, C16, C17, C19, C20, C21, D1, D4, L1, L3, R1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
